File: boards/neurband_c/neurband_c.kicad_sch (KiCad schematic)
At the start: 67 parts, among them J1 FPC 20p 0.5mm (electrode flex), J2 LiPo 3.7V (protected), J3 Charge 5V (magnetic pads), SW1 WAKE / MARK, U1 nRF52832-QFAA, U2 ADS1298IPAGR, U3 XC6206P332MR, U4 TP4054, U5 LSM6DSL, Y1 32MHz 8pF

Commit message: Rev C pre-order rework: analog/RF/DFM fixes, assembly guide and animation
Main board (re-laid out by the layout owner after independent pre-order reviews):
- digital lines (I2C, IMU_INT) moved out of the electrode input field; worst
  coupling 0.89 fF, injected noise <= 0.057 uVrms, P/N mismatch <= 0.71 pF
- local regulator output loop, local ADS/nRF bypassing, C33 at AVDD1, 0603 bulk caps
- RLDIN behind the 100k bias resistor, 10k input arrays (ESD), 12 pF bias RF shunt
- nine tented GND vias in the nRF exposed pad, stitching <= 3 mm in RF/AFE
- footprints carry the fab's 0 deg so the raw position file is correct;
  pin-1/cathode silkscreen, thermal reliefs, 0.5 mm edge pour setback
- DRC 0 / unconnected 0 / parity 0; BOM consolidated to 25 part types

Electrode flex: coverlay closed at the alignment holes, filled stiffener region,
ordering notes; marked not orderable through the rigid-board flow.

Reviews and simulations: analog/noise, on-wrist antenna FDTD (keep the printed
IFA), manufacturing and CPL check against the fab's own footprints.

Mechanics and docs: lead gate, J1 access, snap tolerances; step-by-step build
guide with images and an assembly animation; honest cost update.

Co-Authored-By: Claude Opus 5.5 <noreply@anthropic.com>
Parts:
- added C33: 1uF, Capacitor_SMD:C_0402_1005Metric, symbol Device:C_Small
- added C34: 12pF, Capacitor_SMD:C_0402_1005Metric, symbol Device:C_Small
- C16, C25: value 4.7uF -> 10uF; LCSC C19666 -> C19702; MPN CL10A475KO8NNNC -> CL10A106KP8NNNC
- C28, C6: footprint Capacitor_SMD:C_0402_1005Metric -> Capacitor_SMD:C_0603_1608Metric; LCSC C15525 -> C19702; MPN CL05A106MQ5NUNC -> CL10A106KP8NNNC
- J1: footprint neurband:XUNPU_FPC-05F-20PH20 -> neurband:XUNPU_FPC-05F-20PH20_Centroid
- R10, R9: value 4.7k -> 10k; LCSC C25900 -> C25744; MPN 0402WGF4701TCE -> 0402WGF1002TCE
- RN1, RN2, RN3, RN4: value 4.7k -> 10k; footprint Resistor_SMD:R_Array_Convex_4x0603 -> neurband:R_Array_Convex_4x0603_FabZero; LCSC C1980 -> C29718; MPN 4D03WGJ0472T5E -> 4D03WGJ0103T5E
- U1: footprint Package_DFN_QFN:QFN-48-1EP_6x6mm_P0.4mm_EP4.6x4.6mm -> neurband:QFN-48-1EP_6x6mm_P0.4mm_EP4.6x4.6mm_FabZero
- U2: footprint Package_QFP:TQFP-64_10x10mm_P0.5mm -> neurband:TQFP-64_10x10mm_P0.5mm_FabZero
- U3: footprint Package_TO_SOT_SMD:SOT-23-3 -> neurband:SOT-23-3_FabZero
- U4: footprint Package_TO_SOT_SMD:SOT-23-5 -> neurband:SOT-23-5_FabZero
Connections:
- net +3V3A: now also C33.1
- net BIAS_E: now also C34.1; no longer U2.62 (RLDIN)
- net GND: now also C33.2, C34.2
- net RLD_DRV: now reaches C12.1, R1.1, R2.1, U2.63 (RLDOUT)
- net RLD_DRV: now also U2.62 (RLDIN)
Other:
- note added: "C33: local to AVDD1/AVSS1 (pins 54/53, charge pump)"
- note added: "RN1-RN4: 4x 10 kOhm arrays in series with every electrode (ESD current limit)."
- note added: "VDD: 10uF at pin 48, 100nF at pins 13 and 36"
- note removed: "RN1-RN4: 4x 4.7 kOhm arrays in series with every electrode."
- note removed: "VDD: 4.7uF at pin 48, 100nF at pins 13 and 36"
